Commit message: [kortex_description] Add RS D435 xacro files, and attach to gen3 arm

File: kortex_description/arms/gen3/6dof/urdf/gen3_macro.xacro (robot description, xacro)
@@ -3,4 +3,5 @@
   <!-- Propagate last link name information because it is the gripper's parent link -->
   <xacro:property name="last_arm_link" value="end_effector_link"/>
+  <xacro:include filename="$(find kortex_description)/rs_urdf/_d435.urdf.xacro" />
   <xacro:macro name="load_arm" params="parent:='' dof vision prefix *origin">
     <link name="${prefix}base_link">
@@ -239,3 +240,6 @@
     </joint>
   </xacro:macro>
+  <xacro:sensor_d435 name="rs" topics_ns="camera" parent="${prefix}camera_link" publish_pointcloud="true" use_mesh="true">
+    <origin xyz="-0.0 0.009 -0.009" rpy="0.0 -1.57 1.57"/>
+  </xacro:sensor_d435>
 </robot>

File: kortex_description/arms/gen3/7dof/urdf/gen3_macro.xacro (robot description, xacro)
@@ -3,4 +3,5 @@
   <!-- Propagate last link name information because it is the gripper's parent link -->
   <xacro:property name="last_arm_link" value="end_effector_link"/>
+  <xacro:include filename="$(find kortex_description)/rs_urdf/_d435.urdf.xacro" />
   <xacro:macro name="load_arm" params="parent:='' dof vision prefix *origin">
       <link name="${prefix}base_link">
@@ -329,4 +330,7 @@
         <child  link="${prefix}camera_color_frame" />
       </joint>
+      <xacro:sensor_d435 name="d435" topics_ns="camera" parent="${prefix}camera_link" publish_pointcloud="true" use_mesh="true">
+        <origin xyz="-0.0 0.009 -0.009" rpy="0.0 -1.57 1.57"/>
+      </xacro:sensor_d435>
     </xacro:if>
   </xacro:macro>
