Commit message: Changes required to launch the kortex driver and adapt to the real robot config (testing)

File: kortex_description/robots/gen3_robotiq_2f_85.xacro (robot description, xacro)
@@ -8,5 +8,11 @@
     <xacro:arg name="sim" default="false" />
     <xacro:arg name="prefix" default="" />
-    <xacro:include filename="$(find kortex_description)/robots/kortex_robot.xacro" />
+    <!-- <xacro:include filename="$(find kortex_description)/robots/kortex_robot.xacro" /> -->
+    <xacro:if value="$(arg sim)">
+        <xacro:include filename="$(find kortex_description)/robots/kortex_robot.xacro" />
+    </xacro:if>
+    <xacro:unless value="$(arg sim)">
+        <xacro:include filename="$(find kortex_description)/robots/kortex_robot_real.xacro" />
+    </xacro:unless>
     <xacro:load_robot arm="$(arg arm)" gripper="$(arg gripper)" dof="$(arg dof)" vision="$(arg vision)" sim="$(arg sim)" prefix="$(arg prefix)" />
 </robot>

File: kortex_description/robots/kortex_robot.xacro (robot description, xacro)
@@ -16,13 +16,19 @@
         </xacro:if>
         <!-- Run the macros -->
-        <!-- For gazebo-->
-        <xacro:if value="${sim}">
-            <link name="world" />
-            <joint name="world_to_root" type="fixed">
-                <child link="${prefix}base_link" />
-                <parent link="world" />
-                <origin xyz="0 0 0" rpy="0 0 0" />
-            </joint>
-        </xacro:if>
+        <!-- <!-1- For gazebo-1->-->
+        <!-- <xacro:if value="${sim}">-->
+        <!--     <link name="world" />-->
+        <!--     <joint name="world_to_root" type="fixed">-->
+        <!--         <child link="${prefix}base_link" />-->
+        <!--         <parent link="world" />-->
+        <!--         <origin xyz="0 0 0" rpy="0 0 0" />-->
+        <!--     </joint>-->
+        <!-- </xacro:if>-->
+        <link name="world" />
+        <joint name="world_to_root" type="fixed">
+            <child link="${prefix}base_link" />
+            <parent link="world" />
+            <origin xyz="0 0 0" rpy="0 0 0" />
+        </joint>
         <!-- Load the arm -->
         <xacro:load_arm parent="" dof="${dof}" vision="${vision}" prefix="${prefix}">
