Commit message: Incorporate latest changes required to run on the real robot

File: kortex_description/robots/kortex_robot.xacro (robot description, xacro)
@@ -16,19 +16,19 @@
         </xacro:if>
         <!-- Run the macros -->
-        <!-- <!-1- For gazebo-1->-->
-        <!-- <xacro:if value="${sim}">-->
-        <!--     <link name="world" />-->
-        <!--     <joint name="world_to_root" type="fixed">-->
-        <!--         <child link="${prefix}base_link" />-->
-        <!--         <parent link="world" />-->
-        <!--         <origin xyz="0 0 0" rpy="0 0 0" />-->
-        <!--     </joint>-->
-        <!-- </xacro:if>-->
-        <link name="world" />
-        <joint name="world_to_root" type="fixed">
-            <child link="${prefix}base_link" />
-            <parent link="world" />
-            <origin xyz="0 0 0" rpy="0 0 0" />
-        </joint>
+        <!-- For gazebo-->
+        <xacro:if value="${sim}">
+            <link name="world" />
+            <joint name="world_to_root" type="fixed">
+                <child link="${prefix}base_link" />
+                <parent link="world" />
+                <origin xyz="0 0 0" rpy="0 0 0" />
+            </joint>
+        </xacro:if>
+        <!-- <link name="world" /> -->
+        <!-- <joint name="world_to_root" type="fixed"> -->
+        <!--     <child link="${prefix}base_link" /> -->
+        <!--     <parent link="world" /> -->
+        <!--     <origin xyz="0 0 0" rpy="0 0 0" /> -->
+        <!-- </joint> -->
         <!-- Load the arm -->
         <xacro:load_arm parent="" dof="${dof}" vision="${vision}" prefix="${prefix}">
